File: hardware/power.kicad_sch (KiCad schematic)
At the start: 27 parts, among them J1 USB_B_Micro, J2 battery, U1 WE-TVS-82400102, U2 BQ24075RGT, U3 AMS1117-3.3

Commit message: finish hw development and generate gerber files
Parts:
- removed C10: 0.1u, Capacitor_SMD:C_0402_1005Metric, symbol Device:C
- removed U1: WE-TVS-82400102, Package_TO_SOT_SMD:SOT-23-6, symbol Power_Protection:WE-TVS-82400102
- added U1: DT1446-04V-7, SOT-26-6:SOT95P280X120-6N, symbol RF_Switch:MASWSS0179
- J1: footprint (none) -> Connector_USB:USB_Micro-B_Amphenol_10103594-0001LF_Horizontal
- R1, R2: footprint Resistor_SMD:R_0402_1005Metric -> Resistor_SMD:R_0603_1608Metric
Connections:
- net CONN_D+: now also U1.1 (IO1)
- net CONN_D-: now also U1.4 (IO3)
- net GND: now also U1.2 (VSS)
- net VBUS: now also U1.5 (VCC)
- no-connect marks 5 -> 3
Changed lines of the file:
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@@
   (no_connect (at 182.88 74.93))
   (no_connect (at 182.88 64.77))
-  (no_connect (at 100.33 22.86))
-  (no_connect (at 100.33 27.94))
   (wire (pts (xy 177.8 74.93) (xy 177.8 76.2))
     (stroke (width 0) (type default) (color 0 0 0 0))
@@
     (stroke (width 0) (type default) (color 0 0 0 0))
   )
+  (wire (pts (xy 149.86 21.59) (xy 149.86 22.86))
+    (stroke (width 0) (type default) (color 0 0 0 0))
+  )
   (wire (pts (xy 194.31 101.6) (xy 190.5 101.6))
     (stroke (width 0) (type default) (color 0 0 0 0))
@@
     (stroke (width 0) (type default) (color 0 0 0 0))
   )
-  (wire (pts (xy 102.87 25.4) (xy 102.87 27.94))
-    (stroke (width 0) (type default) (color 0 0 0 0))
-  )
   (wire (pts (xy 116.84 95.25) (xy 116.84 96.52))
     (stroke (width 0) (type default) (color 0 0 0 0))
@@
     (stroke (width 0) (type default) (color 0 0 0 0))
   )
+  (wire (pts (xy 139.7 33.02) (xy 142.24 33.02))
+    (stroke (width 0) (type default) (color 0 0 0 0))
+  )
   (wire (pts (xy 50.8 137.16) (xy 50.8 138.43))
     (stroke (width 0) (type default) (color 0 0 0 0))
@@
     (stroke (width 0) (type default) (color 0 0 0 0))
   )
-  (wire (pts (xy 83.82 25.4) (xy 85.09 25.4))
-    (stroke (width 0) (type default) (color 0 0 0 0))
-  )
   (wire (pts (xy 231.14 90.17) (xy 232.41 90.17))
     (stroke (width 0) (type default) (color 0 0 0 0))
@@
     (stroke (width 0) (type default) (color 0 0 0 0))
   )
-  (wire (pts (xy 256.54 86.36) (xy 256.54 87.63))
+  (wire (pts (xy 149.86 40.64) (xy 149.86 41.91))
     (stroke (width 0) (type default) (color 0 0 0 0))
   )
@@
     (stroke (width 0) (type default) (color 0 0 0 0))
   )
-  (wire (pts (xy 83.82 27.94) (xy 85.09 27.94))
-    (stroke (width 0) (type default) (color 0 0 0 0))
-  )
-  (wire (pts (xy 100.33 25.4) (xy 102.87 25.4))
-    (stroke (width 0) (type default) (color 0 0 0 0))
-  )
   (wire (pts (xy 114.3 54.61) (xy 114.3 60.96))
     (stroke (width 0) (type default) (color 0 0 0 0))
@@
     (stroke (width 0) (type default) (color 0 0 0 0))
   )
+  (wire (pts (xy 157.48 30.48) (xy 158.75 30.48))
+    (stroke (width 0) (type default) (color 0 0 0 0))
+  )
   (wire (pts (xy 40.64 134.62) (xy 41.91 134.62))
     (stroke (width 0) (type default) (color 0 0 0 0))
@@
     (stroke (width 0) (type default) (color 0 0 0 0))
   )
-  (wire (pts (xy 83.82 22.86) (xy 85.09 22.86))
-    (stroke (width 0) (type default) (color 0 0 0 0))
-  )
   (wire (pts (xy 266.7 64.77) (xy 266.7 66.04))
     (stroke (width 0) (type default) (color 0 0 0 0))
   )
-  (wire (pts (xy 256.54 95.25) (xy 256.54 96.52))
-    (stroke (width 0) (type default) (color 0 0 0 0))
-  )
   (wire (pts (xy 266.7 55.88) (xy 266.7 57.15))
     (stroke (width 0) (type default) (color 0 0 0 0))
@@
     (stroke (width 0) (type default) (color 0 0 0 0))
   )
-  (label "VBUS" (at 83.82 25.4 180)
-    (effects (font (size 1.27 1.27)) (justify right bottom))
+  (label "VBUS" (at 149.86 21.59 90)
+    (effects (font (size 1.27 1.27)) (justify left bottom))
   )
   (label "CONN_D+" (at 68.58 43.18 0)
     (effects (font (size 1.27 1.27)) (justify left bottom))
   )
-  (label "CONN_D-" (at 83.82 27.94 180)
+  (label "CONN_D-" (at 139.7 33.02 180)
     (effects (font (size 1.27 1.27)) (justify right bottom))
   )
-  (label "CONN_D+" (at 83.82 22.86 180)
-    (effects (font (size 1.27 1.27)) (justify right bottom))
+  (label "CONN_D+" (at 158.75 30.48 0)
+    (effects (font (size 1.27 1.27)) (justify left bottom))
   )
   (label "VBUS" (at 58.42 38.1 0)
@@
     (effects (font (size 1.27 1.27)) (justify left))
   )
-  (symbol (lib_id "power:+BATT") (at 256.54 86.36 0) (unit 1)
-    (in_bom yes) (on_board yes)
-    (property "Reference" "#PWR020" (id 0) (at 256.54 90.17 0)
-      (effects (font (size 1.27 1.27)) hide)
-    )
-    (property "Value" "+BATT" (id 1) (at 254 82.55 0)
-      (effects (font (size 1.27 1.27)) (justify left))
-    )
-    (property "Footprint" "" (id 2) (at 256.54 86.36 0)
-      (effects (font (size 1.27 1.27)) hide)
-    )
-    (property "Datasheet" "" (id 3) (at 256.54 86.36 0)
-      (effects (font (size 1.27 1.27)) hide)
-    )
-    (pin "1")
-  )
   (symbol (lib_id "power:GND") (at 68.58 59.69 0) (unit 1)
     (in_bom yes) (on_board yes) (fields_autoplaced)
@@
     (property "Reference" "R2" (id 0) (at 81.28 48.26 90))
     (property "Value" "27" (id 1) (at 81.28 45.72 90))
-    (property "Footprint" "Resistor_SMD:R_0402_1005Metric" (id 2) (at 81.28 47.498 90)
+    (property "Footprint" "Resistor_SMD:R_0603_1608Metric" (id 2) (at 81.28 47.498 90)
       (effects (font (size 1.27 1.27)) hide)
     )
@@
     (pin "1")
   )
-  (symbol (lib_id "Device:C") (at 256.54 91.44 0) (unit 1)
-    (in_bom yes) (on_board yes) (fields_autoplaced)
-    (property "Reference" "C10" (id 0) (at 260.35 90.1699 0)
-      (effects (font (size 1.27 1.27)) (justify left))
-    )
-    (property "Value" "0.1u" (id 1) (at 260.35 92.7099 0)
-      (effects (font (size 1.27 1.27)) (justify left))
-    )
-    (property "Footprint" "Capacitor_SMD:C_0402_1005Metric" (id 2) (at 257.5052 95.25 0)
-      (effects (font (size 1.27 1.27)) hide)
-    )
-    (property "Datasheet" "~" (id 3) (at 256.54 91.44 0)
-      (effects (font (size 1.27 1.27)) hide)
-    )
-    (pin "1")
-    (pin "2")
-  )
   (symbol (lib_id "power:GND") (at 114.3 60.96 0) (unit 1)
     (in_bom yes) (on_board yes) (fields_autoplaced)
@@
     (property "Reference" "R1" (id 0) (at 81.28 40.64 90))
     (property "Value" "27" (id 1) (at 81.28 43.18 90))
-    (property "Footprint" "Resistor_SMD:R_0402_1005Metric" (id 2) (at 81.28 44.958 90)
+    (property "Footprint" "Resistor_SMD:R_0603_1608Metric" (id 2) (at 81.28 44.958 90)
       (effects (font (size 1.27 1.27)) hide)
     )
@@
     )
     (property "Datasheet" "" (id 3) (at 256.54 55.88 0)
-      (effects (font (size 1.27 1.27)) hide)
-    )
-    (pin "1")
-  )
-  (symbol (lib_id "power:GND") (at 256.54 96.52 0) (unit 1)
-    (in_bom yes) (on_board yes) (fields_autoplaced)
-    (property "Reference" "#PWR029" (id 0) (at 256.54 102.87 0)
-      (effects (font (size 1.27 1.27)) hide)
-    )
-    (property "Value" "GND" (id 1) (at 256.54 101.6 0))
-    (property "Footprint" "" (id 2) (at 256.54 96.52 0)
-      (effects (font (size 1.27 1.27)) hide)
-    )
-    (property "Datasheet" "" (id 3) (at 256.54 96.52 0)
       (effects (font (size 1.27 1.27)) hide)
     )
@@
     (pin "2")
   )
-  (symbol (lib_id "power:GND") (at 102.87 27.94 0) (unit 1)
-    (in_bom yes) (on_board yes) (fields_autoplaced)
-    (property "Reference" "#PWR01" (id 0) (at 102.87 34.29 0)
-      (effects (font (size 1.27 1.27)) hide)
-    )
-    (property "Value" "GND" (id 1) (at 102.87 33.02 0))
-    (property "Footprint" "" (id 2) (at 102.87 27.94 0)
-      (effects (font (size 1.27 1.27)) hide)
-    )
-    (property "Datasheet" "" (id 3) (at 102.87 27.94 0)
+  (symbol (lib_id "power:GND") (at 149.86 41.91 0) (unit 1)
+    (in_bom yes) (on_board yes) (fields_autoplaced)
+    (property "Reference" "#PWR01" (id 0) (at 149.86 48.26 0)
+      (effects (font (size 1.27 1.27)) hide)
+    )
+    (property "Value" "GND" (id 1) (at 149.86 46.99 0))
+    (property "Footprint" "" (id 2) (at 149.86 41.91 0)
+      (effects (font (size 1.27 1.27)) hide)
+    )
+    (property "Datasheet" "" (id 3) (at 149.86 41.91 0)
       (effects (font (size 1.27 1.27)) hide)
     )
@@
     (pin "2")
   )
-  (symbol (lib_id "Power_Protection:WE-TVS-82400102") (at 92.71 25.4 180) (unit 1)
-    (in_bom yes) (on_board yes) (fields_autoplaced)
-    (property "Reference" "U1" (id 0) (at 91.4399 20.32 90)
-      (effects (font (size 1.27 1.27)) (justify right))
-    )
-    (property "Value" "WE-TVS-82400102" (id 1) (at 93.9799 20.32 90)
-      (effects (font (size 1.27 1.27)) (justify right) hide)
-    )
-    (property "Footprint" "Package_TO_SOT_SMD:SOT-23-6" (id 2) (at 92.71 20.32 0)
-      (effects (font (size 1.27 1.27)) hide)
-    )
-    (property "Datasheet" "https://katalog.we-online.de/pbs/datasheet/82400102.pdf" (id 3) (at 92.71 19.05 0)
+  (symbol (lib_id "RF_Switch:MASWSS0179") (at 152.4 31.75 0) (unit 1)
+    (in_bom yes) (on_board yes)
+    (property "Reference" "U1" (id 0) (at 153.67 24.13 0))
+    (property "Value" "DT1446-04V-7" (id 1) (at 140.97 22.86 0))
+    (property "Footprint" "SOT-26-6:SOT95P280X120-6N" (id 2) (at 153.67 16.51 0)
+      (effects (font (size 1.27 1.27)) hide)
+    )
+    (property "Datasheet" "" (id 3) (at 152.4 29.21 0)
       (effects (font (size 1.27 1.27)) hide)
     )
@@
     (property "Reference" "J1" (id 0) (at 49.53 30.6832 0))
     (property "Value" "USB_B_Micro" (id 1) (at 49.53 33.2232 0))
-    (property "Footprint" "" (id 2) (at 53.34 44.45 0)
-      (effects (font (size 1.27 1.27)) hide)
-    )
+    (property "Footprint" "Connector_USB:USB_Micro-B_Amphenol_10103594-0001LF_Horizontal" (id 2) (at 53.34 44.45 0)
+      (effects (font (size 1.27 1.27)) hide)
+    )
