File: hardware/ucontroller.kicad_sch (KiCad schematic)
At the start: 10 parts, among them Q1 Q_NPN_BEC, Q2 Q_NPN_BEC, SW1 SW_Push, SW2 SW_Push, U4 ESP32-WROOM-32

Commit message: finish hw development and generate gerber files
Connections:
- net SYS_OFF: now also U4.36 (IO22); no longer U4.14 (IO12)
- net TS: now also U4.33 (IO21); no longer U4.13 (IO14)
- net ~{CE}: now also U4.31 (IO19); no longer U4.16 (IO13)
- net ~{CHG}: now also U4.28 (IO17); no longer U4.27 (IO16)
- net ~{PG}: now also U4.30 (IO18); no longer U4.23 (IO15)
- no-connect marks 24 -> 15
Changed lines of the file:
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@@
   (no_connect (at 113.03 85.09))
   (no_connect (at 113.03 87.63))
-  (no_connect (at 143.51 87.63))
-  (no_connect (at 143.51 85.09))
-  (no_connect (at 143.51 90.17))
-  (no_connect (at 143.51 97.79))
   (no_connect (at 143.51 100.33))
   (no_connect (at 143.51 102.87))
@@
   (no_connect (at 143.51 107.95))
   (no_connect (at 143.51 110.49))
-  (no_connect (at 143.51 95.25))
-  (no_connect (at 143.51 92.71))
   (no_connect (at 143.51 59.69))
   (no_connect (at 113.03 62.23))
   (no_connect (at 113.03 59.69))
-  (no_connect (at 143.51 82.55))
-  (no_connect (at 143.51 64.77))
-  (no_connect (at 143.51 67.31))
   (wire (pts (xy 238.76 60.96) (xy 242.57 60.96))
     (stroke (width 0) (type default) (color 0 0 0 0))
@@
     (stroke (width 0) (type default) (color 0 0 0 0))
   )
-  (wire (pts (xy 143.51 72.39) (xy 144.78 72.39))
+  (wire (pts (xy 143.51 87.63) (xy 144.78 87.63))
     (stroke (width 0) (type default) (color 0 0 0 0))
   )
@@
     (stroke (width 0) (type default) (color 0 0 0 0))
   )
+  (wire (pts (xy 144.78 82.55) (xy 143.51 82.55))
+    (stroke (width 0) (type default) (color 0 0 0 0))
+  )
   (wire (pts (xy 242.57 60.96) (xy 242.57 62.23))
     (stroke (width 0) (type default) (color 0 0 0 0))
@@
     (stroke (width 0) (type default) (color 0 0 0 0))
   )
-  (wire (pts (xy 143.51 80.01) (xy 144.78 80.01))
-    (stroke (width 0) (type default) (color 0 0 0 0))
-  )
   (wire (pts (xy 242.57 87.63) (xy 245.11 87.63))
     (stroke (width 0) (type default) (color 0 0 0 0))
@@
     (stroke (width 0) (type default) (color 0 0 0 0))
   )
-  (wire (pts (xy 143.51 69.85) (xy 144.78 69.85))
+  (wire (pts (xy 143.51 92.71) (xy 144.78 92.71))
     (stroke (width 0) (type default) (color 0 0 0 0))
   )
@@
     (stroke (width 0) (type default) (color 0 0 0 0))
   )
+  (wire (pts (xy 143.51 85.09) (xy 144.78 85.09))
+    (stroke (width 0) (type default) (color 0 0 0 0))
+  )
   (wire (pts (xy 212.09 59.69) (xy 215.9 59.69))
     (stroke (width 0) (type default) (color 0 0 0 0))
   )
   (wire (pts (xy 256.54 60.96) (xy 256.54 71.12))
-    (stroke (width 0) (type default) (color 0 0 0 0))
-  )
-  (wire (pts (xy 143.51 77.47) (xy 144.78 77.47))
     (stroke (width 0) (type default) (color 0 0 0 0))
   )
@@
     (stroke (width 0) (type default) (color 0 0 0 0))
   )
-  (wire (pts (xy 143.51 74.93) (xy 144.78 74.93))
+  (wire (pts (xy 143.51 90.17) (xy 144.78 90.17))
     (stroke (width 0) (type default) (color 0 0 0 0))
   )
@@
     (effects (font (size 1.27 1.27)) (justify left bottom))
   )
-  (label "RTS" (at 179.07 85.09 180)
-    (effects (font (size 1.27 1.27)) (justify right bottom))
-  )
   (label "IO0" (at 144.78 54.61 0)
     (effects (font (size 1.27 1.27)) (justify left bottom))
@@
     (effects (font (size 1.27 1.27)) (justify right bottom))
   )
-  (label "DTR" (at 179.07 66.04 180)
-    (effects (font (size 1.27 1.27)) (justify right bottom))
-  )
   (label "IO0" (at 215.9 91.44 0)
     (effects (font (size 1.27 1.27)) (justify left bottom))
@@
     (effects (font (size 1.27 1.27)) (justify left))
   )
-  (hierarchical_label "SYS_OFF" (shape input) (at 144.78 69.85 0)
+  (hierarchical_label "SYS_OFF" (shape input) (at 144.78 92.71 0)
     (effects (font (size 1.27 1.27)) (justify left))
   )
-  (hierarchical_label "TS" (shape input) (at 144.78 74.93 0)
+  (hierarchical_label "TS" (shape input) (at 144.78 90.17 0)
     (effects (font (size 1.27 1.27)) (justify left))
   )
@@
     (effects (font (size 1.27 1.27)) (justify left))
   )
-  (hierarchical_label "~{CHG}" (shape input) (at 144.78 80.01 0)
+  (hierarchical_label "~{CHG}" (shape input) (at 144.78 82.55 0)
     (effects (font (size 1.27 1.27)) (justify left))
   )
-  (hierarchical_label "~{CE}" (shape input) (at 144.78 72.39 0)
+  (hierarchical_label "DTR" (shape input) (at 179.07 66.04 180)
+    (effects (font (size 1.27 1.27)) (justify right))
+  )
+  (hierarchical_label "RTS" (shape input) (at 179.07 85.09 180)
+    (effects (font (size 1.27 1.27)) (justify right))
+  )
+  (hierarchical_label "~{CE}" (shape input) (at 144.78 87.63 0)
     (effects (font (size 1.27 1.27)) (justify left))
   )
-  (hierarchical_label "~{PG}" (shape input) (at 144.78 77.47 0)
+  (hierarchical_label "~{PG}" (shape input) (at 144.78 85.09 0)
     (effects (font (size 1.27 1.27)) (justify left))
   )
