File: hardware/usb.kicad_sch (KiCad schematic)
At the start: 10 parts, among them U5 CP2102N-Axx-xQFN24

Commit message: finish hw development and generate gerber files
Changed lines of the file:
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@@
-    (effects (font (size 1.27 1.27)) (justify left bottom))
-  )
-  (label "RTS" (at 139.7 97.79 0)
-    (effects (font (size 1.27 1.27)) (justify left bottom))
-  )
-  (label "DTR" (at 139.7 105.41 0)
     (effects (font (size 1.27 1.27)) (justify left bottom))
   )
@@
     (effects (font (size 1.27 1.27)) (justify left bottom))
   )
+  (hierarchical_label "DTR" (shape input) (at 139.7 105.41 0)
+    (effects (font (size 1.27 1.27)) (justify left))
+  )
   (hierarchical_label "CP_D+" (shape input) (at 111.76 110.49 180)
     (effects (font (size 1.27 1.27)) (justify right))
@@
     (effects (font (size 1.27 1.27)) (justify right))
   )
+  (hierarchical_label "RTS" (shape input) (at 139.7 97.79 0)
+    (effects (font (size 1.27 1.27)) (justify left))
+  )
   (hierarchical_label "CP_D-" (shape input) (at 111.76 107.95 180)
