File: hardware/wireless.kicad_sch (KiCad schematic)
At the start: 0 parts

Commit message: finish hw development and generate gerber files
Other:
- sheet ucontroller ports: added DTR, RTS; removed none
- sheet usb ports: added DTR, RTS; removed none
Changed lines of the file:
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@@
+    (stroke (width 0) (type default) (color 0 0 0 0))
+  )
+  (wire (pts (xy 162.56 85.09) (xy 184.15 85.09))
     (stroke (width 0) (type default) (color 0 0 0 0))
   )
   (wire (pts (xy 120.65 92.71) (xy 146.05 92.71))
+    (stroke (width 0) (type default) (color 0 0 0 0))
+  )
+  (wire (pts (xy 162.56 87.63) (xy 184.15 87.63))
     (stroke (width 0) (type default) (color 0 0 0 0))
   )
@@
       (effects (font (size 1.27 1.27)) (justify left))
     )
+    (pin "RTS" input (at 162.56 85.09 0)
+      (effects (font (size 1.27 1.27)) (justify right))
+    )
+    (pin "DTR" input (at 162.56 87.63 0)
+      (effects (font (size 1.27 1.27)) (justify right))
+    )
   )
   (sheet (at 184.15 81.28) (size 12.7 27.94) (fields_autoplaced)
@@
       (effects (font (size 1.27 1.27)) (justify left))
     )
+    (pin "RTS" input (at 184.15 85.09 180)
+      (effects (font (size 1.27 1.27)) (justify left))
+    )
+    (pin "DTR" input (at 184.15 87.63 180)
+      (effects (font (size 1.27 1.27)) (justify left))
+    )
   )
   (sheet (at 106.68 81.28) (size 13.97 27.94) (fields_autoplaced)
@@
       (reference "#PWR019") (unit 1) (value "+5V") (footprint "")
     )
-    (path "/576557c4-ef64-4b8f-b30f-1af3610a5c92/022ab15b-c35f-444b-9f25-47cf75638787"
-      (reference "#PWR020") (unit 1) (value "+BATT") (footprint "")
-    )
     (path "/576557c4-ef64-4b8f-b30f-1af3610a5c92/7a501718-3c51-4bb3-816b-25d1b0a62cd9"
       (reference "#PWR021") (unit 1) (value "+BATT") (footprint "")
@@
       (reference "#PWR028") (unit 1) (value "+5V") (footprint "")
     )
-    (path "/576557c4-ef64-4b8f-b30f-1af3610a5c92/2419f776-0a26-481d-af77-8dbd6ff5e20b"
-      (reference "#PWR029") (unit 1) (value "GND") (footprint "")
-    )
     (path "/576557c4-ef64-4b8f-b30f-1af3610a5c92/8a4c1c1f-0f0c-4b15-9f06-9cc10f7f95fe"
       (reference "#PWR030") (unit 1) (value "GND") (footprint "")
@@
       (reference "C9") (unit 1) (value "4.7u") (footprint "Capacitor_SMD:C_0603_1608Metric")
     )
-    (path "/576557c4-ef64-4b8f-b30f-1af3610a5c92/118fb748-7554-4422-be54-07a1e8052010"
-      (reference "C10") (unit 1) (value "0.1u") (footprint "Capacitor_SMD:C_0402_1005Metric")
-    )
     (path "/576557c4-ef64-4b8f-b30f-1af3610a5c92/26f3662b-eadf-454a-bd35-87f470d4058b"
       (reference "C11") (unit 1) (value "0.1u") (footprint "Capacitor_SMD:C_0402_1005Metric")
@@
     )
     (path "/576557c4-ef64-4b8f-b30f-1af3610a5c92/18f35687-2f28-4969-9459-0e9c7ec31065"
-      (reference "R1") (unit 1) (value "27") (footprint "Resistor_SMD:R_0402_1005Metric")
+      (reference "R1") (unit 1) (value "27") (footprint "Resistor_SMD:R_0603_1608Metric")
     )
     (path "/576557c4-ef64-4b8f-b30f-1af3610a5c92/07fc9263-dd91-46fa-83c0-c43e27946e78"
-      (reference "R2") (unit 1) (value "27") (footprint "Resistor_SMD:R_0402_1005Metric")
+      (reference "R2") (unit 1) (value "27") (footprint "Resistor_SMD:R_0603_1608Metric")
     )
     (path "/576557c4-ef64-4b8f-b30f-1af3610a5c92/890ddec2-f71b-43b9-972f-092a534ded6c"
@@
       (reference "SW2") (unit 1) (value "SW_Push") (footprint "Button_Switch_SMD:SW_SPST_B3S-1000")
     )
-    (path "/576557c4-ef64-4b8f-b30f-1af3610a5c92/9edd4323-be0d-4708-8a7e-fba00a204970"
-      (reference "U1") (unit 1) (value "WE-TVS-82400102") (footprint "Package_TO_SOT_SMD:SOT-23-6")
+    (path "/576557c4-ef64-4b8f-b30f-1af3610a5c92/9b2ba8dc-41fa-4029-9058-81810cd563e5"
+      (reference "U1") (unit 1) (value "DT1446-04V-7") (footprint "SOT-26-6:SOT95P280X120-6N")
     )
     (path "/576557c4-ef64-4b8f-b30f-1af3610a5c92/f0bccbda-9d66-422b-8645-9d2ca7aeb6a9"
